File: Project11_He_thong_nha_thong_minh_co_ban/Project11 Schematic.sch (EAGLE design)
At the start: 13 parts, among them U1 ARDUINOR3-BPLACE

Commit message: Cap nhat du an 7,9,11
Parts:
- removed U$1: (no value), DHT11:DHT11
- added R2, R8: 220, SparkFun-Passives:RESISTOR0402-RES
- R7: value 10K -> 220
Connections:
- removed net D7: R7.2, U$1.DATA, U1.D7
- new net N$1: LED3.RED, R2.2
- new net N$2: LED3.GREEN, R6.2
- new net N$3: R5.2
- net D10: now also R6.1; no longer LED3.GREEN
- net D11: now also R2.1; no longer LED3.RED
- net D3: now also R8.1; no longer LED2.GREEN
- net D5: now also R7.1; no longer LED2.RED
- net D9: now also R5.1; no longer LED3.BLUE
- net GND: no longer U$1.GND
- net N$4: now also LED2.RED, R7.2; no longer LED2.VCC, R5.1
- net N$5: now also LED2.BLUE, R8.2; no longer LED3.VCC, R6.1
- net VCC: now also LED2.VCC, LED3.VCC; no longer R5.2, R6.2, R7.1, U$1.VCC
Other:
- moved on the sheet: LED2, LED3, R1, R3, R4, R5, R6, R7, S1

Commit message: Thay doi schematic cua projects.
Connections:
- net D11 renamed N$6
- net D3 renamed N$8
- net D6 renamed N$7
- net N$3: now also LED3.BLUE
Other:
- moved on the sheet: LED2, LED3, R1, R2, R3, R4, R5, R6, R7, R8, S1, SG1
