File: Project7_Bien_tro_dieu_khien_LED_RGB/Project7 Schematic.sch (EAGLE design)
At the start: 8 parts, among them U1 ARDUINOR3-BPLACE

Commit message: Cap nhat du an 7,9,11
Parts:
- removed S1: (no value), adafruit:40-XX
- R1: value 10K -> TRIMPOT-2; device SparkFun-Passives:RESISTOR0402-RES -> SparkFun-Electromechanical:TRIMPOT-2
Connections:
- removed net N$5: R1.2, S1.S1, U1.D2
- new net A0: R1.WIPER, U1.A0
- net GND: now also R1.CCW; no longer S1.P1
- net VCC: now also R1.CW; no longer R1.1
Changed lines of the file:
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@@
 <layer number="223" name="223bmp" color="24" fill="1" visible="no" active="no"/>
 <layer number="224" name="224bmp" color="25" fill="1" visible="no" active="no"/>
+<layer number="225" name="225bmp" color="7" fill="1" visible="yes" active="yes"/>
+<layer number="226" name="226bmp" color="7" fill="1" visible="yes" active="yes"/>
+<layer number="227" name="227bmp" color="7" fill="1" visible="yes" active="yes"/>
+<layer number="228" name="228bmp" color="7" fill="1" visible="yes" active="yes"/>
+<layer number="229" name="229bmp" color="7" fill="1" visible="yes" active="yes"/>
+<layer number="230" name="230bmp" color="7" fill="1" visible="yes" active="yes"/>
 <layer number="231" name="Eagle3D_PG1" color="7" fill="1" visible="no" active="no"/>
 <layer number="232" name="Eagle3D_PG2" color="7" fill="1" visible="no" active="no"/>
@@
 <part name="SUPPLY1" library="SparkFun-Aesthetics" deviceset="VCC" device=""/>
 <part name="GND1" library="SparkFun-Aesthetics" deviceset="GND" device=""/>
-<part name="R1" library="SparkFun-Passives" deviceset="RESISTOR" device="0402-RES" value="10K"/>
 <part name="R2" library="SparkFun-Passives" deviceset="RESISTOR" device="0402-RES" value="220"/>
-<part name="S1" library="adafruit" deviceset="40-XX" device=""/>
 <part name="GND3" library="SparkFun-Aesthetics" deviceset="GND" device=""/>
-<part name="SUPPLY2" library="SparkFun-Aesthetics" deviceset="VCC" device=""/>
 <part name="FRAME1" library="SparkFun-Aesthetics" deviceset="FRAME-LETTER" device=""/>
 <part name="LED1" library="adafruit" deviceset="RGBLED_CA" device="-5MM"/>
@@
 <part name="R4" library="SparkFun-Passives" deviceset="RESISTOR" device="0402-RES" value="220"/>
 <part name="SUPPLY5" library="SparkFun-Aesthetics" deviceset="VCC" device=""/>
+<part name="R1" library="SparkFun-Electromechanical" deviceset="TRIMPOT" device="-2"/>
+<part name="SUPPLY2" library="SparkFun-Aesthetics" deviceset="VCC" device=""/>
+<part name="GND2" library="SparkFun-Aesthetics" deviceset="GND" device=""/>
 </parts>
 <sheets>
@@
 <instance part="SUPPLY1" gate="G$1" x="76.2" y="43.18" rot="R180"/>
 <instance part="GND1" gate="1" x="81.28" y="40.64"/>
-<instance part="R1" gate="G$1" x="99.06" y="119.38"/>
 <instance part="R2" gate="G$1" x="53.34" y="124.46"/>
-<instance part="S1" gate="1" x="114.3" y="121.92" rot="MR270"/>
-<instance part="GND3" gate="1" x="124.46" y="114.3"/>
-<instance part="SUPPLY2" gate="G$1" x="88.9" y="124.46"/>
+<instance part="GND3" gate="1" x="96.52" y="116.84"/>
 <instance part="FRAME1" gate="G$1" x="-33.02" y="-15.24"/>
 <instance part="FRAME1" gate="V" x="114.3" y="-15.24"/>
@@
 <instance part="R4" gate="G$1" x="63.5" y="114.3"/>
 <instance part="SUPPLY5" gate="G$1" x="27.94" y="124.46"/>
+<instance part="R1" gate="R?" x="111.76" y="121.92"/>
+<instance part="SUPPLY2" gate="G$1" x="129.54" y="129.54"/>
+<instance part="GND2" gate="1" x="96.52" y="116.84"/>
 </instances>
 <busses>
@@
 </segment>
 <segment>
-<pinref part="SUPPLY2" gate="G$1" pin="VCC"/>
-<wire x1="88.9" y1="124.46" x2="88.9" y2="119.38" width="0.1524" layer="91"/>
-<pinref part="R1" gate="G$1" pin="1"/>
-<wire x1="88.9" y1="119.38" x2="93.98" y2="119.38" width="0.1524" layer="91"/>
-</segment>
-<segment>
 <pinref part="SUPPLY5" gate="G$1" pin="VCC"/>
 <wire x1="27.94" y1="124.46" x2="27.94" y2="119.38" width="0.1524" layer="91"/>
 <pinref part="LED1" gate="G$1" pin="VCC"/>
+</segment>
+<segment>
+<pinref part="R1" gate="R?" pin="CW"/>
+<wire x1="116.84" y1="121.92" x2="129.54" y2="121.92" width="0.1524" layer="91"/>
+<pinref part="SUPPLY2" gate="G$1" pin="VCC"/>
+<wire x1="129.54" y1="121.92" x2="129.54" y2="129.54" width="0.1524" layer="91"/>
 </segment>
 </net>
@@
 </segment>
 <segment>
-<pinref part="S1" gate="1" pin="P1"/>
 <pinref part="GND3" gate="1" pin="GND"/>
-<wire x1="119.38" y1="119.38" x2="124.46" y2="119.38" width="0.1524" layer="91"/>
-<wire x1="124.46" y1="119.38" x2="124.46" y2="116.84" width="0.1524" layer="91"/>
-</segment>
-</net>
-<net name="N$5" class="0">
-<segment>
-<pinref part="U1" gate="G$1" pin="D2"/>
-<wire x1="93.98" y1="109.22" x2="93.98" y2="114.3" width="0.1524" layer="91"/>
-<pinref part="R1" gate="G$1" pin="2"/>
-<pinref part="S1" gate="1" pin="S1"/>
-<wire x1="104.14" y1="119.38" x2="106.68" y2="119.38" width="0.1524" layer="91"/>
-<wire x1="106.68" y1="119.38" x2="109.22" y2="119.38" width="0.1524" layer="91"/>
-<wire x1="93.98" y1="114.3" x2="106.68" y2="114.3" width="0.1524" layer="91"/>
-<wire x1="106.68" y1="114.3" x2="106.68" y2="119.38" width="0.1524" layer="91"/>
-<junction x="106.68" y="119.38"/>
+<pinref part="GND2" gate="1" pin="GND"/>
+<wire x1="96.52" y1="119.38" x2="96.52" y2="121.92" width="0.1524" layer="91"/>
+<junction x="96.52" y="119.38"/>
+<pinref part="R1" gate="R?" pin="CCW"/>
+<wire x1="96.52" y1="121.92" x2="106.68" y2="121.92" width="0.1524" layer="91"/>
 </segment>
 </net>
@@
 </segment>
 </net>
+<net name="A0" class="0">
+<segment>
+<pinref part="R1" gate="R?" pin="WIPER"/>
+<wire x1="111.76" y1="127" x2="111.76" y2="132.08" width="0.1524" layer="91"/>
+<label x="111.76" y="132.08" size="1.778" layer="95"/>
+</segment>
+<segment>
+<pinref part="U1" gate="G$1" pin="A0"/>
+<wire x1="88.9" y1="48.26" x2="88.9" y2="40.64" width="0.1524" layer="91"/>
+<label x="88.9" y="40.64" size="1.778" layer="95"/>
+</segment>
+</net>

Commit message: Thay doi schematic cua projects.
Connections:
- net A0 renamed N$5
Other:
- moved on the sheet: R1
Changed lines of the file:
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@@
 <?xml version="1.0" encoding="utf-8"?>
 <!DOCTYPE eagle SYSTEM "eagle.dtd">
-<eagle version="7.2.0">
+<eagle version="7.3.0">
 <drawing>
 <settings>
@@
 <instance part="GND1" gate="1" x="81.28" y="40.64"/>
 <instance part="R2" gate="G$1" x="53.34" y="124.46"/>
-<instance part="GND3" gate="1" x="96.52" y="116.84"/>
+<instance part="GND3" gate="1" x="86.36" y="30.48"/>
 <instance part="FRAME1" gate="G$1" x="-33.02" y="-15.24"/>
 <instance part="FRAME1" gate="V" x="114.3" y="-15.24"/>
@@
 <instance part="R4" gate="G$1" x="63.5" y="114.3"/>
 <instance part="SUPPLY5" gate="G$1" x="27.94" y="124.46"/>
-<instance part="R1" gate="R?" x="111.76" y="121.92"/>
-<instance part="SUPPLY2" gate="G$1" x="129.54" y="129.54"/>
-<instance part="GND2" gate="1" x="96.52" y="116.84"/>
+<instance part="R1" gate="R?" x="101.6" y="35.56"/>
+<instance part="SUPPLY2" gate="G$1" x="119.38" y="43.18"/>
+<instance part="GND2" gate="1" x="86.36" y="30.48"/>
 </instances>
 <busses>
@@
 <segment>
 <pinref part="R1" gate="R?" pin="CW"/>
-<wire x1="116.84" y1="121.92" x2="129.54" y2="121.92" width="0.1524" layer="91"/>
+<wire x1="106.68" y1="35.56" x2="119.38" y2="35.56" width="0.1524" layer="91"/>
 <pinref part="SUPPLY2" gate="G$1" pin="VCC"/>
-<wire x1="129.54" y1="121.92" x2="129.54" y2="129.54" width="0.1524" layer="91"/>
+<wire x1="119.38" y1="35.56" x2="119.38" y2="43.18" width="0.1524" layer="91"/>
 </segment>
 </net>
@@
 <pinref part="GND3" gate="1" pin="GND"/>
 <pinref part="GND2" gate="1" pin="GND"/>
-<wire x1="96.52" y1="119.38" x2="96.52" y2="121.92" width="0.1524" layer="91"/>
-<junction x="96.52" y="119.38"/>
+<wire x1="86.36" y1="33.02" x2="86.36" y2="35.56" width="0.1524" layer="91"/>
+<junction x="86.36" y="33.02"/>
 <pinref part="R1" gate="R?" pin="CCW"/>
-<wire x1="96.52" y1="121.92" x2="106.68" y2="121.92" width="0.1524" layer="91"/>
+<wire x1="86.36" y1="35.56" x2="96.52" y2="35.56" width="0.1524" layer="91"/>
 </segment>
 </net>
@@
 </segment>
 </net>
-<net name="A0" class="0">
-<segment>
+<net name="N$5" class="0">
+<segment>
+<pinref part="U1" gate="G$1" pin="A0"/>
+<wire x1="88.9" y1="48.26" x2="88.9" y2="43.18" width="0.1524" layer="91"/>
+<wire x1="88.9" y1="43.18" x2="101.6" y2="43.18" width="0.1524" layer="91"/>
 <pinref part="R1" gate="R?" pin="WIPER"/>
-<wire x1="111.76" y1="127" x2="111.76" y2="132.08" width="0.1524" layer="91"/>
-<label x="111.76" y="132.08" size="1.778" layer="95"/>
-</segment>
-<segment>
-<pinref part="U1" gate="G$1" pin="A0"/>
-<wire x1="88.9" y1="48.26" x2="88.9" y2="40.64" width="0.1524" layer="91"/>
-<label x="88.9" y="40.64" size="1.778" layer="95"/>
-</segment>
-</net>
+<wire x1="101.6" y1="43.18" x2="101.6" y2="40.64" width="0.1524" layer="91"/>
+</segment>
+</net>
